File: pcb/CGMOI/CGMOI.kicad_sch (KiCad schematic)
At the start: 81 parts, among them J1 ADC1E+/-, J10 ActuatorPower12V+/-, J11 MotorPulse/Dir, J12 actuator1Black/Red, J13 actuator2Black/Red, J14 actuator3Black/Red, J15 GyroSCL/SDA, J16 MotorGNDPulse/Dir, J17 Gyro+/-, J2 ADC1A-/+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

Commit message: pcb 2405
Parts:
- J11: value MotorPulse/Dir -> MotorDir/Pulse
Connections:
- net GND: now reaches XA1.GND5 (GND), pin4.1 (pin), pin5.1 (pin), pin6.1 (pin)
- net GND: now also J16.1 (Pin_1), J16.2 (Pin_2), J17.2 (Pin_2), XA1.GND1 (GND), XA1.GND2 (GND), XA1.GND3 (GND), XA1.GND6 (GND), pin10.1 (pin), pin20.1 (pin), pin21.1 (pin), pin22.1 (pin), pin9.1 (pin)
Changed lines of the file:
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@@
 (kicad_sch (version 20211123) (generator eeschema)
   (paper "A4")
+  (junction (at 36.83 89.3572) (diameter 0) (color 0 0 0 0)
+  )
   (junction (at 216.408 34.5948) (diameter 0) (color 0 0 0 0)
   )
+  (junction (at 41.91 90.17) (diameter 0) (color 0 0 0 0)
+  )
   (junction (at 25.4 34.1884) (diameter 0) (color 0 0 0 0)
   )
+  (junction (at 61.976 84.328) (diameter 0) (color 0 0 0 0)
+  )
   (junction (at 124.46 40.7416) (diameter 0) (color 0 0 0 0)
   )
@@
   (junction (at 31.75 34.29) (diameter 0) (color 0 0 0 0)
   )
+  (junction (at 34.29 89.3572) (diameter 0) (color 0 0 0 0)
+  )
   (junction (at 77.47 40.0812) (diameter 0) (color 0 0 0 0)
   )
   (junction (at 25.4 44.958) (diameter 0) (color 0 0 0 0)
   )
+  (junction (at 36.83 89.3064) (diameter 0) (color 0 0 0 0)
+  )
+  (junction (at 52.07 84.328) (diameter 0) (color 0 0 0 0)
+  )
   (junction (at 129.54 40.894) (diameter 0) (color 0 0 0 0)
   )
   (junction (at 71.12 31.8008) (diameter 0) (color 0 0 0 0)
   )
+  (junction (at 39.37 89.3064) (diameter 0) (color 0 0 0 0)
+  )
   (junction (at 31.75 89.3572) (diameter 0) (color 0 0 0 0)
   )
@@
   (junction (at 31.75 68.7324) (diameter 0) (color 0 0 0 0)
   )
+  (junction (at 32.8168 89.3572) (diameter 0) (color 0 0 0 0)
+  )
   (junction (at 255.7272 20.1676) (diameter 0) (color 0 0 0 0)
   )
   (junction (at 71.12 39.8272) (diameter 0) (color 0 0 0 0)
   )
+  (junction (at 39.4208 89.3064) (diameter 0) (color 0 0 0 0)
+  )
   (junction (at 255.6764 35.8648) (diameter 0) (color 0 0 0 0)
+  )
+  (junction (at 54.61 84.328) (diameter 0) (color 0 0 0 0)
   )
   (junction (at 77.47 32.004) (diameter 0) (color 0 0 0 0)
@@
     (stroke (width 0) (type default) (color 0 0 0 0))
   )
+  (wire (pts (xy 61.976 84.328) (xy 62.0268 84.328))
+    (stroke (width 0) (type default) (color 0 0 0 0))
+  )
   (wire (pts (xy 216.662 18.8976) (xy 216.662 25.3492))
     (stroke (width 0) (type default) (color 0 0 0 0))
@@
     (stroke (width 0) (type default) (color 0 0 0 0))
   )
-  (wire (pts (xy 52.07 82.9564) (xy 52.07 88.9))
+  (wire (pts (xy 52.07 82.9564) (xy 52.07 84.328))
     (stroke (width 0) (type default) (color 0 0 0 0))
   )
@@
     (stroke (width 0) (type default) (color 0 0 0 0))
   )
-  (wire (pts (xy 54.61 82.9564) (xy 54.61 90.17))
+  (wire (pts (xy 54.61 82.9564) (xy 54.61 84.328))
     (stroke (width 0) (type default) (color 0 0 0 0))
   )
@@
     (stroke (width 0) (type default) (color 0 0 0 0))
   )
+  (wire (pts (xy 41.91 90.17) (xy 41.91 91.44))
+    (stroke (width 0) (type default) (color 0 0 0 0))
+  )
   (wire (pts (xy 64.77 184.15) (xy 64.77 187.96))
     (stroke (width 0) (type default) (color 0 0 0 0))
@@
     (stroke (width 0) (type default) (color 0 0 0 0))
   )
+  (wire (pts (xy 36.83 89.3572) (xy 36.83 91.44))
+    (stroke (width 0) (type default) (color 0 0 0 0))
+  )
   (wire (pts (xy 174.498 108.9152) (xy 177.7492 108.9152))
     (stroke (width 0) (type default) (color 0 0 0 0))
@@
     (stroke (width 0) (type default) (color 0 0 0 0))
   )
-  (wire (pts (xy 32.8168 89.3572) (xy 31.75 89.3572))
+  (wire (pts (xy 31.75 89.3572) (xy 32.8168 89.3572))
     (stroke (width 0) (type default) (color 0 0 0 0))
   )
@@
     (stroke (width 0) (type default) (color 0 0 0 0))
   )
+  (wire (pts (xy 36.83 89.3064) (xy 36.83 89.3572))
+    (stroke (width 0) (type default) (color 0 0 0 0))
+  )
+  (wire (pts (xy 54.61 84.328) (xy 61.976 84.328))
+    (stroke (width 0) (type default) (color 0 0 0 0))
+  )
   (wire (pts (xy 174.3456 98.1456) (xy 175.6156 98.1456))
     (stroke (width 0) (type default) (color 0 0 0 0))
@@
     (stroke (width 0) (type default) (color 0 0 0 0))
   )
+  (wire (pts (xy 54.61 84.328) (xy 54.61 90.17))
+    (stroke (width 0) (type default) (color 0 0 0 0))
+  )
   (wire (pts (xy 77.47 22.352) (xy 77.47 32.004))
     (stroke (width 0) (type default) (color 0 0 0 0))
@@
     (stroke (width 0) (type default) (color 0 0 0 0))
   )
+  (wire (pts (xy 32.8168 89.3572) (xy 34.29 89.3572))
+    (stroke (width 0) (type default) (color 0 0 0 0))
+  )
   (wire (pts (xy 60.8076 163.322) (xy 60.8076 166.2176))
     (stroke (width 0) (type default) (color 0 0 0 0))
@@
     (stroke (width 0) (type default) (color 0 0 0 0))
   )
+  (wire (pts (xy 54.61 84.328) (xy 52.07 84.328))
+    (stroke (width 0) (type default) (color 0 0 0 0))
+  )
   (wire (pts (xy 173.1264 32.8676) (xy 176.022 32.8676))
     (stroke (width 0) (type default) (color 0 0 0 0))
@@
     (stroke (width 0) (type default) (color 0 0 0 0))
   )
+  (wire (pts (xy 39.4208 89.3064) (xy 41.91 89.3064))
+    (stroke (width 0) (type default) (color 0 0 0 0))
+  )
   (wire (pts (xy 107.95 72.6948) (xy 107.95 91.44))
     (stroke (width 0) (type default) (color 0 0 0 0))
   )
+  (wire (pts (xy 34.29 89.3572) (xy 34.29 91.44))
+    (stroke (width 0) (type default) (color 0 0 0 0))
+  )
   (wire (pts (xy 255.7272 20.1676) (xy 255.7272 26.8224))
     (stroke (width 0) (type default) (color 0 0 0 0))
@@
     (stroke (width 0) (type default) (color 0 0 0 0))
   )
+  (wire (pts (xy 34.29 89.3572) (xy 36.83 89.3572))
+    (stroke (width 0) (type default) (color 0 0 0 0))
+  )
   (wire (pts (xy 97.79 157.48) (xy 97.79 162.5092))
     (stroke (width 0) (type default) (color 0 0 0 0))
@@
     (stroke (width 0) (type default) (color 0 0 0 0))
   )
+  (wire (pts (xy 36.83 89.3064) (xy 39.37 89.3064))
+    (stroke (width 0) (type default) (color 0 0 0 0))
+  )
   (wire (pts (xy 220.0656 130.3528) (xy 220.0656 134.3152))
     (stroke (width 0) (type default) (color 0 0 0 0))
@@
     (stroke (width 0) (type default) (color 0 0 0 0))
   )
-  (wire (pts (xy 41.91 90.17) (xy 41.91 91.44))
+  (wire (pts (xy 41.91 89.3064) (xy 41.91 90.17))
     (stroke (width 0) (type default) (color 0 0 0 0))
   )
@@
     (stroke (width 0) (type default) (color 0 0 0 0))
   )
-  (wire (pts (xy 34.29 86.36) (xy 34.29 91.44))
+  (wire (pts (xy 34.29 86.36) (xy 34.29 89.3572))
     (stroke (width 0) (type default) (color 0 0 0 0))
   )
@@
     (stroke (width 0) (type default) (color 0 0 0 0))
   )
-  (wire (pts (xy 39.37 88.9) (xy 39.37 91.44))
+  (wire (pts (xy 39.37 88.9) (xy 39.37 89.3064))
     (stroke (width 0) (type default) (color 0 0 0 0))
   )
@@
     (stroke (width 0) (type default) (color 0 0 0 0))
   )
+  (wire (pts (xy 39.37 89.3064) (xy 39.37 91.44))
+    (stroke (width 0) (type default) (color 0 0 0 0))
+  )
   (wire (pts (xy 39.37 157.48) (xy 39.37 166.37))
     (stroke (width 0) (type default) (color 0 0 0 0))
@@
     (stroke (width 0) (type default) (color 0 0 0 0))
   )
+  (wire (pts (xy 52.07 84.328) (xy 52.07 88.9))
+    (stroke (width 0) (type default) (color 0 0 0 0))
+  )
   (wire (pts (xy 258.5212 130.3528) (xy 258.5212 134.874))
     (stroke (width 0) (type default) (color 0 0 0 0))
@@
     (stroke (width 0) (type default) (color 0 0 0 0))
   )
-  (wire (pts (xy 36.83 87.63) (xy 36.83 91.44))
+  (wire (pts (xy 36.83 87.63) (xy 36.83 89.3064))
     (stroke (width 0) (type default) (color 0 0 0 0))
   )
@@
   (symbol (lib_id "Connector:Screw_Terminal_01x02") (at 127.254 169.5704 270) (unit 1)
     (in_bom yes) (on_board yes) (fields_autoplaced)
-    (property "Reference" "J11" (id 0) (at 130.4544 168.3003 90)
-      (effects (font (size 1.27 1.27)) (justify left))
-    )
-    (property "Value" "MotorPulse/Dir" (id 1) (at 130.4544 170.8403 90)
+    (property "Reference" "J11" (id 0) (at 129.54 168.3003 90)
+      (effects (font (size 1.27 1.27)) (justify left))
+    )
+    (property "Value" "MotorDir/Pulse" (id 1) (at 129.54 170.8403 90)
       (effects (font (size 1.27 1.27)) (justify left))
     )
@@
     (pin "1")
   )
+  (symbol (lib_id "power:GND") (at 61.976 84.328 90) (unit 1)
+    (in_bom yes) (on_board yes) (fields_autoplaced)
+    (property "Reference" "#PWR?" (id 0) (at 68.326 84.328 0)
+      (effects (font (size 1.27 1.27)) hide)
+    )
+    (property "Value" "GND" (id 1) (at 66.04 84.3279 90)
+      (effects (font (size 1.27 1.27)) (justify right))
+    )
+    (property "Footprint" "" (id 2) (at 61.976 84.328 0)
+      (effects (font (size 1.27 1.27)) hide)
+    )
+    (property "Datasheet" "" (id 3) (at 61.976 84.328 0)
+      (effects (font (size 1.27 1.27)) hide)
+    )
+    (pin "1")
+  )
   (symbol (lib_id "cgmoi:pin") (at 256.794 141.478 180) (unit 1)
     (in_bom yes) (on_board yes)
@@
   )
   (symbol_instances
+    (path "/fb8f1790-cda5-4111-8cbc-a71001a6b06e"
+      (reference "#PWR?") (unit 1) (value "GND") (footprint "")
+    )
     (path "/07058de7-f688-454c-bfbe-7df82a190fcd"
       (reference "J1") (unit 1) (value "ADC1E+/-") (footprint "cgmoi:screw terminal")
@@
     )
     (path "/13afc725-3e1c-440d-8c7f-80c6b37a5ceb"
-      (reference "J11") (unit 1) (value "MotorPulse/Dir") (footprint "cgmoi:screw terminal")
+      (reference "J11") (unit 1) (value "MotorDir/Pulse") (footprint "cgmoi:screw terminal")
     )
     (path "/e334f9fb-52ab-4885-9edd-f10e1388af58"
