File: pcb/CGMOI/CGMOI.kicad_pcb (KiCad board)
At the start: 2 copper layers, 170 x 155 mm, 81 parts, among them J1 ADC1E+/-, J10 ActuatorPower12V+/-, J11 MotorPulse/Dir, J12 actuator1Black/Red, J13 actuator2Black/Red, J14 actuator3Black/Red, J15 GyroSCL/SDA, J16 MotorGNDPulse/Dir, J17 Gyro+/-, J2 ADC1A-/+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

Commit message: pcb1905
Routing:
- net Net-(J17-Pad1): track 67.7 -> 85.7 mm, vias 0 -> 2
- net Net-(XA1-PadGND3): track 212.1 -> 223.8 mm, vias 6 -> 10
- net Net-(XA1-PadGND5): track 145.8 -> 151.6 mm
- net Net-(J10-Pad2): track 323.7 -> 318.6 mm
- net Net-(J14-Pad2): track 108.4 -> 104.2 mm
- net Net-(J12-Pad2): track 92.6 -> 88.6 mm
- net Net-(XA1-Pad5V1): track 236.8 -> 240.4 mm, vias 6 -> 10
- net Net-(J14-Pad1): track 110.8 -> 114.0 mm
- net Net-(XA1-Pad5V3): track 150.9 -> 153.9 mm
- net Net-(XA1-PadD32): track 82.6 -> 85.3 mm
- net Net-(J13-Pad2): track 98.3 -> 97.2 mm
- net Net-(XA1-PadD41): track 103.7 -> 103.3 mm, vias 6 -> 4
- net Net-(XA1-PadD42): vias 8 -> 4
- net Net-(XA1-PadD45): vias 10 -> 6
- net Net-(XA1-PadD44): vias 10 -> 6
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
Commit message: pcb 2405
Parts:
- J11: value MotorPulse/Dir -> MotorDir/Pulse
- moved J15 3.23 mm to (29.1, 30.7)
- moved J17 2.78 mm to (29.2, 41.2)
- moved J11 2.54 mm to (29.2, 51.4)
- moved XA1 2.51 mm to (21.4, 115.7)
- moved J16 2.16 mm to (29.2, 61.9)
- moved J3 1.96 mm to (60.0, 37.0)
- moved J10 1.84 mm to (29.2, 72.2)
- moved J6 1.82 mm to (108.2, 37.2)
- moved J9 1.72 mm to (83.7, 37.2)
- moved J12 1.33 mm to (102.5, 79.8)
- moved J2 1.09 mm to (60.0, 47.9)
- moved J5 1.05 mm to (108.2, 48.0)
- moved J8 1.00 mm to (83.7, 47.9)
- moved J13 0.70 mm to (102.5, 90.4)
- moved pin57 0.44 mm to (183.9, 39.6)
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Connections:
- J16 pad 1: Net-(J16-Pad1) -> GND
- J16 pad 2: Net-(J16-Pad2) -> GND
- J17 pad 2: Net-(J17-Pad2) -> GND
- XA1 pad GND1: Net-(J16-Pad2) -> GND
- XA1 pad GND2: Net-(J16-Pad1) -> GND
- XA1 pad GND3: Net-(XA1-PadGND3) -> GND
- XA1 pad GND5: Net-(XA1-PadGND5) -> GND
- XA1 pad GND6: Net-(J17-Pad2) -> GND
- pin10 pad 1: Net-(J17-Pad2) -> GND
- pin20 pad 1: Net-(XA1-PadGND3) -> GND
- pin21 pad 1: Net-(XA1-PadGND3) -> GND
- pin22 pad 1: Net-(XA1-PadGND3) -> GND
- pin4 pad 1: Net-(XA1-PadGND5) -> GND
- pin5 pad 1: Net-(XA1-PadGND5) -> GND
- pin6 pad 1: Net-(XA1-PadGND5) -> GND
- pin9 pad 1: Net-(J17-Pad2) -> GND
Routing:
- net GND: track 0.00 -> 803.0 mm, vias 0 -> 700
- net Net-(XA1-PadGND3): track 223.8 -> 0.00 mm, vias 10 -> 0
- net Net-(J17-Pad2): track 199.6 -> 0.00 mm, vias 2 -> 0
- net Net-(XA1-PadGND5): track 151.6 -> 0.00 mm, vias 8 -> 0
- net Net-(J16-Pad2): track 116.5 -> 0.00 mm
- net Net-(J16-Pad1): track 90.3 -> 0.00 mm, vias 2 -> 0
- net Net-(J2-Pad1): track 140.4 -> 154.6 mm
- net Net-(J3-Pad1): track 149.3 -> 141.8 mm
- net Net-(J11-Pad1): track 131.3 -> 137.6 mm
- net Net-(J11-Pad2): track 134.2 -> 139.4 mm
- net Net-(J17-Pad1): track 85.7 -> 90.5 mm
- net Net-(J15-Pad2): track 222.0 -> 226.0 mm
- net Net-(XA1-PadD45): track 134.3 -> 137.2 mm
- net Net-(XA1-PadD22): track 100.2 -> 102.7 mm
- net Net-(XA1-Pad5V1): track 240.4 -> 242.9 mm
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- added copper zone on B.Cu, net GND
- added copper zone on F.Cu, net GND
Other:
- board text added: "A+(G)"
- board text added: "A-(W)"
- board text added: "E+(R)"
- board text added: "E-(B)"
- board text added: "Red1"
- board text removed: "A+"
- board text removed: "A-"
- board text removed: "E+"
- board text removed: "E-"
- board text removed: "RED1"

Commit message: final pcb with gerbe file
Parts:
- added G***: LOGO, cgmoi:NuSpace KiCad Logo, F.Cu at (143.3, 167.5)
- moved J10 1.00 mm to (29.2, 73.2)
- moved J11 1.00 mm to (29.2, 52.4)
- moved J15 1.00 mm to (29.1, 31.7)
- moved J16 1.00 mm to (29.2, 62.9)
- moved J17 1.00 mm to (29.2, 42.2)
Routing:
- net Net-(J2-Pad1): track 154.6 -> 143.4 mm
- net Net-(J11-Pad1): track 137.6 -> 135.8 mm
- net GND: track 803.0 -> 804.6 mm, vias 700 -> 782
- net Net-(J15-Pad2): track 226.0 -> 224.4 mm
- net Net-(J17-Pad1): track 90.5 -> 89.5 mm
- net Net-(J15-Pad1): track 229.6 -> 228.7 mm
Other:
- board text added: "The HW V1"
